File: PCB /array.kicad_pcb (KiCad board)
At the start: 2 copper layers, 8 parts

Commit message: asd
Parts:
- added REF**: SOT-23_DIO, FDA:SOT-23_DIO, F.Cu at (161.6, 87.8)
- added REF**: SOT-23_DIO, FDA:SOT-23_DIO, F.Cu at (151.5, 67.5)
- added REF**: SOT-23_DIO, FDA:SOT-23_DIO, F.Cu at (110.8, 87.8)
- added REF**: SOT-23_DIO, FDA:SOT-23_DIO, F.Cu at (131.2, 57.3)
- added REF**: SOT-23_DIO, FDA:SOT-23_DIO, F.Cu at (141.3, 118.3)
- added REF**: SIP-21, FDA:SIP-21, F.Cu at (97.5, 86.5)
- added REF**: SOT-23_DIO, FDA:SOT-23_DIO, F.Cu at (131.2, 87.8)
- added REF**: SOT-23_DIO, FDA:SOT-23_DIO, F.Cu at (161.6, 118.3)
- added REF**: SOT-23_DIO, FDA:SOT-23_DIO, F.Cu at (110.8, 118.3)
- added REF**: SOT-23_DIO, FDA:SOT-23_DIO, F.Cu at (100.7, 87.8)
- added REF**: SOT-23_DIO, FDA:SOT-23_DIO, F.Cu at (151.5, 77.7)
- added REF**: SOT-23_DIO, FDA:SOT-23_DIO, F.Cu at (121.0, 118.3)
- added REF**: SOT-23_DIO, FDA:SOT-23_DIO, F.Cu at (121.0, 77.7)
- added REF**: SOT-23_DIO, FDA:SOT-23_DIO, F.Cu at (110.8, 67.5)
- added REF**: SOT-23_DIO, FDA:SOT-23_DIO, F.Cu at (100.7, 57.4)
- added REF**: SOT-23_DIO, FDA:SOT-23_DIO, F.Cu at (110.8, 108.2)
- added REF**: SOT-23_DIO, FDA:SOT-23_DIO, F.Cu at (121.0, 87.8)
- added REF**: SOT-23_DIO, FDA:SOT-23_DIO, F.Cu at (110.8, 77.7)
- added REF**: SOT-23_DIO, FDA:SOT-23_DIO, F.Cu at (100.7, 98.0)
- added REF**: SOT-23_DIO, FDA:SOT-23_DIO, F.Cu at (141.3, 67.5)
- added REF**: SOT-23_DIO, FDA:SOT-23_DIO, F.Cu at (141.3, 57.3)
- added REF**: SOT-23_DIO, FDA:SOT-23_DIO, F.Cu at (141.3, 108.1)
- added REF**: SOT-23_DIO, FDA:SOT-23_DIO, F.Cu at (121.0, 98.0)
- added REF**: SOT-23_DIO, FDA:SOT-23_DIO, F.Cu at (161.6, 98.0)
- added REF**: SOT-23_DIO, FDA:SOT-23_DIO, F.Cu at (141.3, 77.7)
- added REF**: SOT-23_DIO, FDA:SOT-23_DIO, F.Cu at (121.0, 67.5)
- added REF**: SOT-23_DIO, FDA:SOT-23_DIO, F.Cu at (161.6, 67.5)
- added REF**: SOT-23_DIO, FDA:SOT-23_DIO, F.Cu at (141.3, 87.8)
- added REF**: SOT-23_DIO, FDA:SOT-23_DIO, F.Cu at (100.7, 67.5)
- added REF**: SOT-23_DIO, FDA:SOT-23_DIO, F.Cu at (110.8, 57.4)
- added REF**: SOT-23_DIO, FDA:SOT-23_DIO, F.Cu at (161.6, 77.7)
- added REF**: SOT-23_DIO, FDA:SOT-23_DIO, F.Cu at (131.2, 67.5)
- added REF**: SOT-23_DIO, FDA:SOT-23_DIO, F.Cu at (131.2, 77.7)
- added REF**: SOT-23_DIO, FDA:SOT-23_DIO, F.Cu at (141.3, 98.0)
- added REF**: SOT-23_DIO, FDA:SOT-23_DIO, F.Cu at (110.8, 98.0)
- added REF**: SOT-23_DIO, FDA:SOT-23_DIO, F.Cu at (131.2, 98.0)
- added REF**: SOT-23_DIO, FDA:SOT-23_DIO, F.Cu at (151.5, 87.8)
- added REF**: SOT-23_DIO, FDA:SOT-23_DIO, F.Cu at (121.0, 108.1)
- added REF**: SOT-23_DIO, FDA:SOT-23_DIO, F.Cu at (151.5, 57.3)
- added REF**: SOT-23_DIO, FDA:SOT-23_DIO, F.Cu at (121.0, 57.3)
- added REF**: SOT-23_DIO, FDA:SOT-23_DIO, F.Cu at (151.5, 98.0)
- added REF**: SOT-23_DIO, FDA:SOT-23_DIO, F.Cu at (161.6, 108.1)
- added REF**: SOT-23_DIO, FDA:SOT-23_DIO, F.Cu at (131.2, 118.3)
- added REF**: SOT-23_DIO, FDA:SOT-23_DIO, F.Cu at (100.7, 77.7)
- added REF**: SOT-23_DIO, FDA:SOT-23_DIO, F.Cu at (161.6, 57.3)
- added REF**: SOT-23_DIO, FDA:SOT-23_DIO, F.Cu at (151.5, 118.3)
- added REF**: SOT-23_DIO, FDA:SOT-23_DIO, F.Cu at (131.2, 108.1)
- added REF**: SOT-23_DIO, FDA:SOT-23_DIO, F.Cu at (151.5, 108.1)
- added REF**: SOT-23_DIO, FDA:SOT-23_DIO, F.Cu at (100.7, 108.2)
- moved REF** 56.8 mm to (100.7, 118.3), turned to 90 degrees
- moved REF** 4.17 mm to (97.7, 89.4)
- moved REF** 4.17 mm to (158.6, 89.4)
- moved REF** 4.17 mm to (148.4, 89.4)
- moved REF** 4.17 mm to (138.2, 89.4)
- moved REF** 4.17 mm to (107.8, 89.4)
- moved REF** 4.17 mm to (118.0, 89.4)
- moved REF** 4.17 mm to (128.1, 89.4)
Routing:
- net (no net): track 0.00 -> 1636.6 mm
Other:
- board text added: "+on -off"
- board text added: "-on +off"

Commit message: asd
Parts:
- moved REF** 30.4 mm to (127.8, 89.1)
Routing:
- net (no net): track 1636.6 -> 1883.7 mm
Other:
- board outline added: 76.2 x 76.2 mm

Commit message: asd
Parts:
- removed the REF** at (127.8, 89.1)
- added REF**: SIP-22, FDA:SIP-22, F.Cu at (127.8, 90.4)
Routing:
- added copper zone on B.Cu, net (none)
Other:
- board text added: "7x7 Test Flipdot Array, Designed in 2024 by Tyler Bowers"
- board text added: "ABCD"
