File: controller pcb/array.kicad_pcb (KiCad board)
At the start: 4 copper layers, 28 parts

Commit message: asd
Parts:
- added REF**: CAPRR254W54L381T254H466, FDA:10uf cap, F.Cu at (93.9, 125.1)
- added REF**: CAPRR254W54L381T254H466, FDA:10uf cap, F.Cu at (155.2, 147.6)
- added REF**: 0ZCG_BEL, FDA:0ZCG_BEL, F.Cu at (216.0, 128.1)
- added REF**: CAPRR254W54L381T254H466, FDA:10uf cap, F.Cu at (144.7, 128.0)
- added REF**: CAPRR254W54L381T254H466, FDA:10uf cap, F.Cu at (205.3, 102.7)
- added REF**: RPI Zero2w, FDA:RPI Zero2w, F.Cu at (87.2, 125.2)
- added REF**: CAPRR254W54L381T254H466, FDA:10uf cap, F.Cu at (93.8, 149.5)
- added REF**: CUI_PJ-002A, FDA:CUI_PJ-002A, F.Cu at (216.0, 136.4)
- added REF**: CAPRR254W54L381T254H466, FDA:10uf cap, F.Cu at (144.7, 102.8)
- added REF**: R-78C/E-1.0_SIP3_11.6X8.5X10.4_RCP, FDA:R78E5, F.Cu at (213.1, 106.1)
- added REF**: CAPRR254W54L381T254H466, FDA:10uf cap, F.Cu at (155.2, 122.4)
- moved REF** 32.8 mm to (205.3, 127.9)
Routing:
- net (no net): track 2512.8 -> 3392.5 mm
Other:
- board text added: "TBD62783APG -> high side TBD62381APG -> low side"

Commit message: asd
Parts:
- removed the REF** at (93.9, 125.1)
- removed the REF** at (28.2, 86.0)
- removed the REF** at (104.3, 149.2)
- removed the REF** at (96.4, 127.8)
- removed the REF** at (104.3, 124.4)
- removed the REF** at (93.8, 149.5)
- removed the REF** at (216.0, 136.4)
- removed the REF** at (213.1, 106.1)
- removed the REF** at (96.4, 103.0)
- added REF**: R78E5-FD, FDA:R78E5-FD, F.Cu at (215.6, 112.8)
- added REF**: CAPRR254W54L381T254H466, FDA:10uf cap, F.Cu at (94.3, 122.4)
- added REF**: CAP_YX_5X11_RUB, FDA:CAP_YX_5X11_RUB, F.Cu at (215.8, 106.1)
- added REF**: SN74AHC595N, Luminator:SN74AHC595N, F.Cu at (96.8, 100.3)
- added REF**: 8x10k R Array, Luminator:8x10 R Array, F.Cu at (104.6, 121.7)
- added REF**: 8x10k R Array, Luminator:8x10 R Array, F.Cu at (104.6, 146.4)
- added REF**: CAPRR254W54L381T254H466, FDA:10uf cap, F.Cu at (94.3, 147.6)
- added REF**: SN74AHC595N, Luminator:SN74AHC595N, F.Cu at (96.8, 125.1)
- added REF**: CAP, FDA:CAP_YX_10X16_RUB, F.Cu at (210.3, 118.8)
- added REF**: PJ-002A-F, FDA:PJ-002A-F, F.Cu at (201.0, 101.6)
- REF** (x4): value TBD62873APG -> TBD62783APG
- moved REF** 17.7 mm to (210.0, 111.5)
- moved REF** 11.4 mm to (194.0, 101.3), turned to 180 degrees
- moved REF** 2.76 mm to (108.7, 126.1)
- moved REF** 2.76 mm to (108.7, 101.3)
- moved REF** 0.93 mm to (144.7, 103.7)
Routing:
- net (no net): track 3392.5 -> 4774.1 mm, vias 85 -> 86
- added copper zone on B.Cu, net (none)
Other:
- board outline added: 133.7 x 51.2 mm
- board text added: "+5v"
- board text added: "1"
- board text added: "12v Barrel"
- board text added: "ESP32"
- board text added: "Flipdot Array Controller Tyler Bowers 2024"
